File: ClockWork.kicad_pcb (KiCad board)
At the start: 2 copper layers, 73.7 x 140.3 mm, 65 parts, among them J1 Conn_02x01_Row_Letter_First, J10 Conn_01x04_Male, J11 Conn_01x04_Male, J12 Conn_01x04_Female, J13 Conn_01x04_Male, J14 Conn_01x04_Female, J15 Conn_02x01_Row_Letter_First, J16 Conn_01x02_Female, J2 USB_A, J3 Conn_01x03_Male, J4 Conn_01x03_Female, J5 Conn_01x06_Male, J6 Conn_01x06_Female, J7 Conn_01x04_Female, J8 Conn_01x04_Male, J9 Conn_01x04_Female, SW1 SW_SPDT, SW2 SW_Push, SW3 SW_Push, SW4 SW_Push, SW5 SW_Push, U1 4520, U10 4520, U11 4056, U12 4011, U13 4056, U2 4011, U3 4520, U4 4056, U5 4001, U6 4011, U7 4011, U8 4056, U9 4011, Y1 Crystal

Commit message: Minor changes in design
Routing:
- added copper zone on F.Cu, net (none)
Changed lines of the file:
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@@
     (property "Sheetname" "")
     (attr through_hole)
-    (fp_text reference "J15" (at -3.175 0 180) (layer "F.SilkS")
+    (fp_text reference "J15" (at 0 5.08 180) (layer "F.SilkS")
       (effects (font (size 1 1) (thickness 0.15)))
     )
@@
     )
   )
+  (zone (net 0) (net_name "") (layer "F.Cu") (hatch edge 0.508)
+    (connect_pads (clearance 0.508))
+    (min_thickness 0.254) (filled_areas_thickness no)
+    (fill yes (thermal_gap 0.508) (thermal_bridge_width 0.508))
+    (polygon
+      (pts
+        (xy 158.75 81.28)
+        (xy 157.48 81.28)
+        (xy 157.48 83.82)
+        (xy 160.02 83.82)
+        (xy 160.02 82.55)
+        (xy 161.29 82.55)
+        (xy 161.29 85.09)
+        (xy 160.02 86.36)
+        (xy 160.02 85.09)
+        (xy 156.21 85.09)
+        (xy 156.21 81.28)
+        (xy 154.94 81.28)
+        (xy 156.21 80.01)
+        (xy 158.75 80.01)
+      )
+    )
+  )
+  (zone (net 0) (net_name "") (layer "F.Cu") (hatch edge 0.508)
+    (connect_pads (clearance 0.508))
+    (min_thickness 0.254) (filled_areas_thickness no)
+    (fill yes (thermal_gap 0.508) (thermal_bridge_width 0.508))
+    (polygon
+      (pts
+        (xy 166.37 114.935)
+        (xy 165.1 114.935)
+        (xy 165.1 117.475)
+        (xy 167.64 117.475)
+        (xy 167.64 116.205)
+        (xy 168.91 116.205)
+        (xy 168.91 118.745)
+        (xy 167.64 120.015)
+        (xy 167.64 118.745)
+        (xy 163.83 118.745)
+        (xy 163.83 114.935)
+        (xy 162.56 114.935)
+        (xy 163.83 113.665)
+        (xy 166.37 113.665)
+      )
+    )
+  )
+  (zone (net 0) (net_name "") (layer "F.Cu") (hatch edge 0.508)
+    (connect_pads (clearance 0.508))
+    (min_thickness 0.254) (filled_areas_thickness no)
+    (fill yes (thermal_gap 0.508) (thermal_bridge_width 0.508))
+    (polygon
+      (pts
+        (xy 161.29 81.28)
+        (xy 160.02 81.28)
+        (xy 160.02 80.01)
+        (xy 161.29 80.01)
+      )
+    )
+  )
+  (zone (net 0) (net_name "") (layer "F.Cu") (hatch edge 0.508)
+    (connect_pads (clearance 0.508))
+    (min_thickness 0.254) (filled_areas_thickness no)
+    (fill yes (thermal_gap 0.508) (thermal_bridge_width 0.508))
+    (polygon
+      (pts
+        (xy 168.91 114.935)
+        (xy 167.64 114.935)
+        (xy 167.64 113.665)
+        (xy 168.91 113.665)
+      )
+    )
+  )
   (zone (net 129) (net_name "/GND_buttons") (layer "B.Cu") (hatch edge 0.508)
     (connect_pads (clearance 0.508))
@@
       )
     )
+  )
+  (zone (net 0) (net_name "") (layer "B.Cu") (hatch edge 0.508)
+    (connect_pads (clearance 0))
+    (min_thickness 0.254)
+    (keepout (tracks not_allowed) (vias not_allowed) (pads not_allowed) (copperpour not_allowed) (footprints allowed))
+    (fill (thermal_gap 0.508) (thermal_bridge_width 0.508))
+    (polygon
+      (pts
+        (xy 148.59 170.18)
+        (xy 147.955 170.18)
+        (xy 147.955 171.45)
+        (xy 149.225 171.45)
+        (xy 149.225 170.815)
+        (xy 149.86 170.815)
+        (xy 149.86 172.085)
+        (xy 149.225 172.72)
+        (xy 149.225 172.085)
+        (xy 147.955 172.085)
+        (xy 147.32 172.085)
+        (xy 147.32 170.18)
+        (xy 146.685 170.18)
+        (xy 147.32 169.545)
+        (xy 148.59 169.545)
+      )
+    )
+  )
+  (zone (net 0) (net_name "") (layer "B.Cu") (hatch edge 0.508)
+    (connect_pads (clearance 0))
+    (min_thickness 0.254)
+    (keepout (tracks not_allowed) (vias not_allowed) (pads not_allowed) (copperpour not_allowed) (footprints allowed))
+    (fill (thermal_gap 0.508) (thermal_bridge_width 0.508))
+    (polygon
+      (pts
+        (xy 166.37 155.575)
+        (xy 165.735 155.575)
+        (xy 165.735 156.845)
+        (xy 167.005 156.845)
+        (xy 167.005 156.21)
+        (xy 167.64 156.21)
+        (xy 167.64 157.48)
+        (xy 167.005 158.115)
+        (xy 167.005 157.48)
+        (xy 165.735 157.48)
+        (xy 165.1 157.48)
+        (xy 165.1 155.575)
+        (xy 164.465 155.575)
+        (xy 165.1 154.94)
+        (xy 166.37 154.94)
+      )
+    )
+  )
+  (zone (net 0) (net_name "") (layer "B.Cu") (hatch edge 0.508)
+    (connect_pads (clearance 0))
+    (min_thickness 0.254)
+    (keepout (tracks not_allowed) (vias not_allowed) (pads not_allowed) (copperpour not_allowed) (footprints allowed))
+    (fill (thermal_gap 0.508) (thermal_bridge_width 0.508))
+    (polygon
+      (pts
+        (xy 149.86 170.18)
+        (xy 149.225 170.18)
+        (xy 149.225 169.545)
+        (xy 149.86 169.545)
+      )
+    )
+  )
+  (zone (net 0) (net_name "") (layer "B.Cu") (hatch edge 0.508)
+    (connect_pads (clearance 0))
+    (min_thickness 0.254)
+    (keepout (tracks not_allowed) (vias not_allowed) (pads not_allowed) (copperpour not_allowed) (footprints allowed))
+    (fill (thermal_gap 0.508) (thermal_bridge_width 0.508))
+    (polygon
+      (pts
+        (xy 167.64 155.575)
+        (xy 167.005 155.575)
+        (xy 167.005 154.94)
+        (xy 167.64 154.94)
+      )
+    )
